File: kicad/ida-button/4gates.kicad_pcb (KiCad board)
At the start: 2 copper layers, 84 x 100 mm, 80 parts, among them J1 PANEL_SOCKET, J10 CV_OUT, J11 GATE_OUT, J12 TRIG_OUT, J13 PANEL_HEADER_B, J2 CV_IN, J3 CV_OUT, J4 EURO_PWR_2x5, J5 GATE_OUT, J6 TRIG_OUT, J7 PANEL_HEADER, J8 PANEL_SOCKET, J9 CV_IN, Q1 J113, Q10 BC547, Q11 BC557, Q2 BC547, Q3 BC547, Q7 BC557, Q8 J113, Q9 BC547, SW1 SW_SPDT, SW2 SW_SPDT, SW3 ARCADE_BTN, SW4 ARCADE_BTN_B, U1 TL074, U2 40106, U4 TL074

Commit message: stylophone rev1
Parts:
- removed Q10, Q2, Q3, Q9: BC547, Package_TO_SOT_THT:TO-92_Inline
- removed Q11, Q7: BC557, Package_TO_SOT_THT:TO-92_Inline
- removed R31, R34, R38, R39, R41: 1k, PCM_4ms_Resistor:R_Axial_DIN0207_L6.3mm_D2.5mm_P7.62mm_Horizontal
- removed R32, R36: 100k, PCM_4ms_Resistor:R_Axial_DIN0207_L6.3mm_D2.5mm_P7.62mm_Horizontal
- removed R37: R, PCM_4ms_Resistor:R_Axial_DIN0207_L6.3mm_D2.5mm_P7.62mm_Horizontal
- removed R40: 47k, PCM_4ms_Resistor:R_Axial_DIN0207_L6.3mm_D2.5mm_P7.62mm_Horizontal
- added C10: 0.1uf, PCM_4ms_Capacitor:C_Disc_P5.08mm, F.Cu at (115.3, 78.5)
- added C11: 0.1uf, PCM_4ms_Capacitor:C_Disc_P5.08mm, F.Cu at (113.1, 92.8)
- added C12: 0.1uf, PCM_4ms_Capacitor:C_Disc_P5.08mm, F.Cu at (112.8, 106.8)
- added C13: 0.1uf, PCM_4ms_Capacitor:C_Disc_P5.08mm, F.Cu at (118.2, 122.1)
- added C14: 10nf, PCM_4ms_Capacitor:C_Disc_P5.08mm, F.Cu at (115.3, 75.3)
- added C5: 0.1uf, PCM_4ms_Capacitor:C_Disc_P5.08mm, F.Cu at (124.4, 68.6)
- added C6: 0.33uf, PCM_4ms_Capacitor:C_Disc_P5.08mm, F.Cu at (124.6, 77.3)
- added C7: 10nf, PCM_4ms_Capacitor:C_Disc_P5.08mm, F.Cu at (115.9, 127.6)
- added C9: 0.1uf, PCM_4ms_Capacitor:C_Disc_P5.08mm, F.Cu at (105.2, 92.8)
- added D6: D, PCM_4ms_Diode:D_DO-35_P7.62mm_Horizontal, F.Cu at (105.7, 73.7)
- added J14: PANEL_A_IN, Connector_PinSocket_2.54mm:PinSocket_1x05_P2.54mm_Vertical, B.Cu at (152.8, 136.3)
- added J15: PANEL_B_OUT, Connector_PinSocket_2.54mm:PinSocket_1x05_P2.54mm_Vertical, B.Cu at (182.0, 52.0)
- added J16: B_IN, Connector_PinHeader_2.54mm:PinHeader_1x05_P2.54mm_Vertical, F.Cu at (102.7, 52.3)
- added J17: B_OUT, Connector_PinHeader_2.54mm:PinHeader_1x05_P2.54mm_Vertical, F.Cu at (132.2, 52.5)
- added U3: L78L05_TO92, Package_TO_SOT_THT:TO-92_Inline, F.Cu at (123.6, 71.6)
- D1: value D_Zener -> D; footprint Diode_THT:D_DO-35_SOD27_P7.62mm_Horizontal -> PCM_4ms_Diode:D_DO-35_P7.62mm_Horizontal
- D3, D4: footprint Diode_THT:D_DO-41_SOD81_P10.16mm_Horizontal -> PCM_4ms_Diode:D_DO-41_P7.62mm_Horizontal
- J1: value PANEL_SOCKET -> A_OUT; footprint Connector_PinHeader_2.54mm:PinHeader_2x05_P2.54mm_Vertical -> Connector_PinHeader_2.54mm:PinHeader_1x05_P2.54mm_Vertical; moved to F.Cu
- J13: value PANEL_HEADER_B -> PANEL_B_IN; footprint Connector_PinHeader_2.54mm:PinHeader_2x05_P2.54mm_Vertical -> Connector_PinSocket_2.54mm:PinSocket_1x05_P2.54mm_Vertical; moved to B.Cu
- J4: footprint Connector_PinHeader_2.54mm:PinHeader_2x05_P2.54mm_Vertical -> KitsBlips:Pins_2x05_2.54mm_TH_Europower_shrouded
- J7: value PANEL_HEADER -> A_IN; footprint Connector_PinHeader_2.54mm:PinHeader_2x05_P2.54mm_Vertical -> Connector_PinHeader_2.54mm:PinHeader_1x05_P2.54mm_Vertical
- J8: value PANEL_SOCKET -> PANEL_A_OUT; footprint Connector_PinHeader_2.54mm:PinHeader_2x05_P2.54mm_Vertical -> Connector_PinSocket_2.54mm:PinSocket_1x05_P2.54mm_Vertical
- R10, R12: value 100k -> 20k
- R11, R9: value 1k -> 20k
- R14: value 47k -> 1k
- R21, R22, R30, R33, R35, R8: value 1k -> 100k
- R3: value 10k -> 1k
- R7: value R -> 1k
- SW3, SW4: footprint Connector_PinHeader_2.54mm:PinHeader_1x02_P2.54mm_Horizontal -> Connector_JST:JST_XH_S2B-XH-A-1_1x02_P2.50mm_Horizontal; moved to B.Cu
- moved R15 131.7 mm to (179.0, 126.7), turned to 90 degrees
- moved R28 130.5 mm to (180.8, 70.0), turned to -90 degrees
- moved R13 127.1 mm to (181.6, 126.7), turned to -90 degrees
- moved R23 121.4 mm to (178.1, 70.0), turned to -90 degrees
- moved R14 108.6 mm to (155.6, 126.6), turned to 90 degrees
- moved R7 103.7 mm to (152.1, 70.0), turned to 90 degrees
- moved R19 91.7 mm to (154.8, 70.0), turned to 90 degrees
- moved J8 87.0 mm to (181.8, 136.5)
- moved R35 86.3 mm to (124.7, 62.6), turned to 0 degrees
- moved R30 82.7 mm to (124.7, 65.2), turned to 180 degrees
- moved R16 81.5 mm to (132.2, 128.5), turned to -90 degrees
- moved C1 79.9 mm to (129.3, 129.4), turned to 90 degrees
- moved Q1 79.8 mm to (119.2, 138.0), turned to -90 degrees
- moved C4 79.8 mm to (123.8, 57.1)
- moved R26 78.8 mm to (124.8, 51.6), turned to 0 degrees
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Connections:
- net Net-(R35-Pad2) renamed /B/B_TRIG_OUT
- net Net-(U2-Pad10) renamed /B/B_BUTTON_NONINV
- net Net-(U4C--) renamed /B/B_CV_OUT
- C1 pad 2: /A/BUTTON_XOR -> /A/A_BUTTON_XOR
- C4 pad 2: /B/BUTTON_XOR -> /B/B_BUTTON_XOR
- D1 pad 1: +5V -> Net-(D1-K)
- D1 pad 2: GND1 -> Net-(D1-A)
- J1 pad 1: GND2 -> /A/A_BUTTON_INV
- J1 pad 2: /front_panel/POT_1 -> /A/A_BUTTON_NONINV
- J1 pad 3: Net-(J1-Pin_3) -> /A/A_CV_OUT
- J1 pad 4: Net-(J1-Pin_4) -> /A/A_TRIG_OUT
- J1 pad 5: Net-(J1-Pin_5) -> /A/A_BUTTON_XOR
- J10 pad T: Net-(J8-Pin_4) -> Net-(J10-PadT)
- J11 pad T: Net-(J8-Pin_6) -> Net-(J11-PadT)
- J12 pad T: Net-(J8-Pin_8) -> Net-(J12-PadT)
- J13 pad 1: GND1 -> GND2
- J13 pad 2: /B/CV_IN_PIN -> GND2
- J13 pad 3: /B/TOGGLE_OUT -> /front_panel/B_ATTENUATOR_INV
- J13 pad 4: /B/CV_OUT_PIN -> /front_panel/B_ATTENUATOR_NONINV
- J13 pad 5: +5V -> /front_panel/B_BUTTON_XOR
- J2 pad T: /front_panel/POT_1 -> /front_panel/A_ATTENUATOR_INV
- J3 pad T: Net-(J1-Pin_4) -> Net-(J3-PadT)
- J5 pad T: Net-(J1-Pin_6) -> Net-(J5-PadT)
- J6 pad T: Net-(J1-Pin_8) -> Net-(J6-PadT)
- J7 pad 1: GND1 -> +5V
- J7 pad 2: /A/CV_IN_PIN -> +5V
- J7 pad 3: /A/TOGGLE_OUT -> /A/A_ATTENUATOR_INV
- J7 pad 4: /A/CV_OUT_PIN -> /A/A_ATTENUATOR_NONINV
- J7 pad 5: +5V -> /A/A_BUTTON_XOR
- J8 pad 1: GND2 -> /front_panel/A_BUTTON_INV
- J8 pad 2: Net-(J8-Pin_2) -> /front_panel/A_BUTTON_NONINV
- J8 pad 3: Net-(J8-Pin_3) -> /front_panel/A_CV_OUT
- J8 pad 4: Net-(J8-Pin_4) -> /front_panel/A_TRIG_OUT
- J8 pad 5: Net-(J8-Pin_5) -> /front_panel/A_GATE_OUT
- J9 pad T: Net-(J8-Pin_2) -> /front_panel/B_ATTENUATOR_INV
- J9 pad TN: unconnected-(J9-PadTN) -> Net-(J9-PadTN)
- R1 pad 1: /A/CV_IN_PIN -> /A/A_ATTENUATOR_INV
- R10 pad 1: Net-(Q3-E) -> Net-(D1-A)
- R10 pad 2: Net-(Q2-B) -> Net-(D1-K)
- R11 pad 1: /A/TOGGLE_OUT -> +5V
- R11 pad 2: GND1 -> Net-(D6-A)
- R12 pad 1: /A/TOGGLE_OUT -> Net-(D6-A)
- R12 pad 2: Net-(Q3-B) -> Net-(D6-K)
- R13 pad 1: /A/CV_OUT_PIN -> /front_panel/A_GATE_OUT
- R13 pad 2: Net-(U1C--) -> Net-(J5-PadT)
- R14 pad 1: Net-(Q2-C) -> Net-(J3-PadT)
- R14 pad 2: Net-(Q7-B) -> /front_panel/A_CV_OUT
- R15 pad 1: Net-(Q7-C) -> /front_panel/A_TRIG_OUT
- R15 pad 2: GND1 -> Net-(J6-PadT)
- R16 pad 1: /A/BUTTON_XOR -> /A/A_BUTTON_XOR
- R19 pad 1: Net-(R19-Pad1) -> Net-(J10-PadT)
- R19 pad 2: Net-(R17-Pad2) -> /front_panel/B_CV_OUT
- R20 pad 1: /B/CV_IN_PIN -> /B/B_ATTENUATOR_INV
- R22 pad 2: Net-(R22-Pad2) -> /A/A_TRIG_OUT
- R23 pad 1: Net-(R22-Pad2) -> /front_panel/B_GATE_OUT
- R23 pad 2: /A/TRIG_OUT_PIN -> Net-(J11-PadT)
- R24 pad 1: /B/BUTTON_XOR -> /B/B_BUTTON_XOR
- R28 pad 1: Net-(R28-Pad1) -> /front_panel/B_TRIG_OUT
- R28 pad 2: Net-(R25-Pad2) -> Net-(J12-PadT)
- R3 pad 1: +12V -> /front_panel/IN_5V
- R3 pad 2: +5V -> unconnected-(J2-PadTN)
- R7 pad 1: /A/BUTTON_XOR -> /front_panel/IN_5V
- R7 pad 2: /A/GATE_OUT_PIN -> Net-(J9-PadTN)
- R9 pad 1: GND1 -> +5V
- R9 pad 2: Net-(Q3-E) -> Net-(D1-A)
- RV1 pad 1: /front_panel/POT_1 -> GND2
- RV1 pad 2: Net-(J1-Pin_9) -> /front_panel/A_ATTENUATOR_NONINV
- RV1 pad 3: GND2 -> /front_panel/A_ATTENUATOR_INV
- RV2 pad 1: Net-(J8-Pin_7) -> GND2
- RV2 pad 2: Net-(J8-Pin_9) -> /front_panel/B_ATTENUATOR_NONINV
- RV2 pad 3: GND2 -> /front_panel/B_ATTENUATOR_INV
- SW1 pad 1: unconnected-(SW1-A-Pad1) -> /front_panel/A_BUTTON_NONINV
- SW1 pad 2: Net-(J1-Pin_5) -> /front_panel/A_BUTTON_XOR
- SW1 pad 3: Net-(J1-Pin_3) -> /front_panel/A_BUTTON_INV
- SW2 pad 1: unconnected-(SW2-A-Pad1) -> /front_panel/B_BUTTON_NONINV
- SW2 pad 2: Net-(J8-Pin_5) -> /front_panel/B_BUTTON_XOR
- SW2 pad 3: Net-(J8-Pin_3) -> /front_panel/B_BUTTON_INV
- SW3 pad 1: +5V -> GND1
- SW3 pad 2: Net-(Q3-E) -> Net-(D1-A)
- SW4 pad 1: +5V -> GND1
- SW4 pad 2: Net-(Q10-E) -> Net-(D6-A)
- U1 pad 14: Net-(R22-Pad2) -> /A/A_TRIG_OUT
- U1 pad 3: /A/POT_2 -> /A/A_ATTENUATOR_NONINV
- U1 pad 6: /A/BUTTON_XOR -> /A/A_BUTTON_XOR
- U1 pad 8: Net-(U1C--) -> /A/A_CV_OUT
- U1 pad 9: Net-(U1C--) -> /A/A_CV_OUT
- U2 pad 1: Net-(Q7-C) -> Net-(D1-K)
- U2 pad 11: Net-(Q11-C) -> Net-(D6-K)
- U2 pad 12: /B/BUTTON_XOR -> /B/B_BUTTON_INV
- U2 pad 2: Net-(U2-Pad2) -> /A/A_BUTTON_NONINV
- U2 pad 3: Net-(U2-Pad2) -> /A/A_BUTTON_NONINV
- U2 pad 4: /A/BUTTON_XOR -> /A/A_BUTTON_INV
- U2 pad 5: Net-(R19-Pad1) -> Net-(R17-Pad2)
- U2 pad 9: Net-(R28-Pad1) -> Net-(R25-Pad2)
- U4 pad 3: /B/POT_2 -> /B/B_ATTENUATOR_NONINV
- U4 pad 6: /B/BUTTON_XOR -> /B/B_BUTTON_XOR
Routing:
- net +5V: track 0.00 -> 114.4 mm, vias 0 -> 5
- net +12V: track 0.00 -> 90.9 mm, vias 0 -> 4
- net /A/A_BUTTON_XOR: track 0.00 -> 78.1 mm, vias 0 -> 3
- net +2.5V: track 0.00 -> 76.8 mm, vias 0 -> 3
- net /B/B_BUTTON_INV: track 0.00 -> 75.8 mm, vias 0 -> 4
- net /B/B_BUTTON_XOR: track 0.00 -> 73.8 mm, vias 0 -> 3
- net /B/B_BUTTON_NONINV: track 0.00 -> 68.5 mm, vias 0 -> 2
- net /front_panel/IN_5V: track 0.00 -> 66.4 mm
- net -12V: track 0.00 -> 62.6 mm, vias 0 -> 1
- net /A/A_TRIG_OUT: track 0.00 -> 60.4 mm, vias 0 -> 2
- net Net-(R25-Pad2): track 0.00 -> 60.4 mm, vias 0 -> 3
- net /A/A_BUTTON_NONINV: track 0.00 -> 60.1 mm, vias 0 -> 2
- net /front_panel/A_BUTTON_NONINV: track 0.00 -> 55.4 mm, vias 0 -> 1
- net /front_panel/A_BUTTON_INV: track 0.00 -> 54.8 mm, vias 0 -> 1
- net /A/A_BUTTON_INV: track 0.00 -> 53.8 mm, vias 0 -> 1
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- added copper zone on B.Cu, net GND1
- added copper zone on F.Cu, net GND1
- added copper zone on B.Cu, net GND2
- added copper zone on F.Cu, net GND2
