File: kicad/ida-button/B.kicad_sch (KiCad schematic)
At the start: 29 parts, among them J13 PANEL_HEADER_B, Q10 BC547, Q11 BC557, Q8 J113, Q9 BC547, SW4 ARCADE_BTN_B, U2 40106, U4 TL074

Commit message: stylophone rev1
Parts:
- removed J13: PANEL_HEADER_B, Connector_PinHeader_2.54mm:PinHeader_2x05_P2.54mm_Vertical, symbol Connector_Generic:Conn_02x05_Odd_Even
- removed Q10, Q9: BC547, Package_TO_SOT_THT:TO-92_Inline, symbol Transistor_BJT:BC547
- removed Q11: BC557, Package_TO_SOT_THT:TO-92_Inline, symbol Transistor_BJT:BC557
- removed R28, R31, R34, R38, R39, R41: 1k, PCM_4ms_Resistor:R_Axial_DIN0207_L6.3mm_D2.5mm_P7.62mm_Horizontal, symbol Device:R
- removed R32, R36: 100k, PCM_4ms_Resistor:R_Axial_DIN0207_L6.3mm_D2.5mm_P7.62mm_Horizontal, symbol Device:R
- removed R37: R, PCM_4ms_Resistor:R_Axial_DIN0207_L6.3mm_D2.5mm_P7.62mm_Horizontal, symbol Device:R
- removed R40: 47k, PCM_4ms_Resistor:R_Axial_DIN0207_L6.3mm_D2.5mm_P7.62mm_Horizontal, symbol Device:R
- added C14: 10nf, PCM_4ms_Capacitor:C_Disc_P5.08mm, symbol Device:C
- added D6: D, PCM_4ms_Diode:D_DO-35_P7.62mm_Horizontal, symbol Device:D
- added R11, R12: 20k, PCM_4ms_Resistor:R_Axial_DIN0207_L6.3mm_D2.5mm_P7.62mm_Horizontal, symbol Device:R
- R30, R33, R35: value 1k -> 100k
- SW4: footprint Connector_PinHeader_2.54mm:PinHeader_1x02_P2.54mm_Horizontal -> Connector_JST:JST_XH_S2B-XH-A-1_1x02_P2.50mm_Horizontal
Connections:
- net +5V: now also R11.1; no longer SW4.1
- net GND1: now also SW4.1, C14.2
- net B_BUTTON_NONINV: now reaches U2.10, U2.13
- net at U2.11: now also C14.1, D6.1 (K), R12.2
- net at SW4.2: now also D6.2 (A), R11.2, R12.1
- net at R25.2, R26.2: now also U2.9
- net B_TRIG_OUT: now reaches R35.2, U4.14
- net B_CV_OUT: now reaches U4.8, U4.9 (-)
- net BUTTON_XOR renamed B_BUTTON_XOR
- net B_BUTTON_XOR: no longer U2.12
- net CV_IN_PIN renamed B_ATTENUATOR_INV
- net POT_2 renamed B_ATTENUATOR_NONINV
- new net B_BUTTON_INV: U2.12
Other:
- note added: "TODO: breadboard to find ideal debounce values"
- moved on the sheet: D5, Q8, R20, R27, R29, R33, SW4, U2E, U2F, U4A, U4B, U4C
