File: kicad/ida-button/front_panel.kicad_sch (KiCad schematic)
At the start: 20 parts, among them J10 CV_OUT, J11 GATE_OUT, J12 TRIG_OUT, J2 CV_IN, J3 CV_OUT, J5 GATE_OUT, J6 TRIG_OUT, J9 CV_IN, SW1 SW_SPDT, SW2 SW_SPDT

Commit message: been a minute huh
Parts:
- renumbered R31 to R?
Changed lines of the file:
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@@
 		(dnp no)
 		(fields_autoplaced yes)
-		(property "Reference" "R31"
+		(property "Reference" "R?"
 			(at 111.76 16.51 90)
 			(effects
@@
 		(pin "2"
 		)
-		(instances)
+		(instances
+			(project "4gates"
+				(path "/373e077e-bfc7-40f9-b9b8-adde168d27e9/f765f6b7-0977-4652-ae5d-8c5e5aa74b64"
+					(reference "R?")
+					(unit 1)
+				)
+			)
+		)
 	)
 	(symbol
