File: kicad/ida-button-smt/A.kicad_sch (KiCad schematic)
At the start: 19 parts, among them Q1 J113, SW3 ARCADE_BTN, U1 TL074, U2 40106

Commit message: stylophone rev1
Parts:
- C1, C7: footprint PCM_4ms_Capacitor:C_Disc_P5.08mm -> Capacitor_SMD:C_0603_1608Metric
- D1, D2: footprint PCM_4ms_Diode:D_DO-35_P7.62mm_Horizontal -> Diode_SMD:D_0603_1608Metric
- Q1: footprint Package_TO_SOT_THT:TO-92 -> Package_TO_SOT_SMD:SOT-23_Handsoldering
- R1, R10, R16, R17, R18, R2, R21, R22, R5, R8, R9: footprint PCM_4ms_Resistor:R_Axial_DIN0207_L6.3mm_D2.5mm_P7.62mm_Horizontal -> Resistor_SMD:R_0603_1608Metric
- U1: footprint Package_DIP:DIP-14_W7.62mm_Socket -> Package_SO:SSOP-14_5.3x6.2mm_P0.65mm
- U2: footprint Package_DIP:DIP-14_W7.62mm_Socket -> Package_SO:TSSOP-14_4.4x5mm_P0.65mm
Changed lines of the file:
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@@
 			)
 		)
-		(property "Footprint" "PCM_4ms_Resistor:R_Axial_DIN0207_L6.3mm_D2.5mm_P7.62mm_Horizontal"
+		(property "Footprint" "Resistor_SMD:R_0603_1608Metric"
 			(at 57.15 178.308 90)
 			(effects
@@
 			)
 		)
-		(property "Footprint" "Package_DIP:DIP-14_W7.62mm_Socket"
+		(property "Footprint" "Package_SO:SSOP-14_5.3x6.2mm_P0.65mm"
 			(at 111.76 171.45 0)
 			(effects
@@
 			)
 		)
-		(property "Footprint" "Package_DIP:DIP-14_W7.62mm_Socket"
+		(property "Footprint" "Package_SO:SSOP-14_5.3x6.2mm_P0.65mm"
 			(at 116.84 105.41 0)
 			(effects
@@
 			)
 		)
-		(property "Footprint" "PCM_4ms_Resistor:R_Axial_DIN0207_L6.3mm_D2.5mm_P7.62mm_Horizontal"
+		(property "Footprint" "Resistor_SMD:R_0603_1608Metric"
 			(at 60.452 26.67 90)
 			(effects
@@
 			)
 		)
-		(property "Footprint" "PCM_4ms_Resistor:R_Axial_DIN0207_L6.3mm_D2.5mm_P7.62mm_Horizontal"
+		(property "Footprint" "Resistor_SMD:R_0603_1608Metric"
 			(at 114.808 121.92 90)
 			(effects
@@
 			)
 		)
-		(property "Footprint" "PCM_4ms_Resistor:R_Axial_DIN0207_L6.3mm_D2.5mm_P7.62mm_Horizontal"
+		(property "Footprint" "Resistor_SMD:R_0603_1608Metric"
 			(at 95.25 144.018 90)
 			(effects
@@
 			)
 		)
-		(property "Footprint" "Package_DIP:DIP-14_W7.62mm_Socket"
+		(property "Footprint" "Package_SO:TSSOP-14_4.4x5mm_P0.65mm"
 			(at 114.3 43.18 0)
 			(effects
@@
 			)
 		)
-		(property "Footprint" "PCM_4ms_Diode:D_DO-35_P7.62mm_Horizontal"
+		(property "Footprint" "Diode_SMD:D_0603_1608Metric"
 			(at 68.58 31.75 0)
 			(effects
@@
 			)
 		)
-		(property "Footprint" "PCM_4ms_Resistor:R_Axial_DIN0207_L6.3mm_D2.5mm_P7.62mm_Horizontal"
+		(property "Footprint" "Resistor_SMD:R_0603_1608Metric"
 			(at 68.58 44.958 90)
 			(effects
@@
 			)
 		)
-		(property "Footprint" "PCM_4ms_Capacitor:C_Disc_P5.08mm"
+		(property "Footprint" "Capacitor_SMD:C_0603_1608Metric"
 			(at 75.8952 50.8 0)
 			(effects
@@
 			)
 		)
-		(property "Footprint" "PCM_4ms_Capacitor:C_Disc_P5.08mm"
+		(property "Footprint" "Capacitor_SMD:C_0603_1608Metric"
 			(at 46.99 177.4952 0)
 			(effects
@@
 			)
 		)
-		(property "Footprint" "PCM_4ms_Resistor:R_Axial_DIN0207_L6.3mm_D2.5mm_P7.62mm_Horizontal"
+		(property "Footprint" "Resistor_SMD:R_0603_1608Metric"
 			(at 131.572 144.78 90)
 			(effects
@@
 			)
 		)
-		(property "Footprint" "PCM_4ms_Resistor:R_Axial_DIN0207_L6.3mm_D2.5mm_P7.62mm_Horizontal"
+		(property "Footprint" "Resistor_SMD:R_0603_1608Metric"
 			(at 72.39 132.588 90)
 			(effects
@@
 			)
 		)
-		(property "Footprint" "PCM_4ms_Diode:D_DO-35_P7.62mm_Horizontal"
+		(property "Footprint" "Diode_SMD:D_0603_1608Metric"
 			(at 125.73 114.3 0)
 			(effects
@@
 			)
 		)
-		(property "Footprint" "Package_DIP:DIP-14_W7.62mm_Socket"
+		(property "Footprint" "Package_SO:SSOP-14_5.3x6.2mm_P0.65mm"
 			(at 93.98 125.73 0)
 			(effects
@@
 			)
 		)
-		(property "Footprint" "Package_DIP:DIP-14_W7.62mm_Socket"
+		(property "Footprint" "Package_SO:TSSOP-14_4.4x5mm_P0.65mm"
 			(at 81.28 176.53 0)
 			(effects
@@
 			)
 		)
-		(property "Footprint" "PCM_4ms_Resistor:R_Axial_DIN0207_L6.3mm_D2.5mm_P7.62mm_Horizontal"
+		(property "Footprint" "Resistor_SMD:R_0603_1608Metric"
 			(at 92.71 178.308 90)
 			(effects
@@
 			)
 		)
-		(property "Footprint" "PCM_4ms_Resistor:R_Axial_DIN0207_L6.3mm_D2.5mm_P7.62mm_Horizontal"
+		(property "Footprint" "Resistor_SMD:R_0603_1608Metric"
 			(at 64.008 184.15 90)
 			(effects
@@
 			)
 		)
-		(property "Footprint" "Package_DIP:DIP-14_W7.62mm_Socket"
+		(property "Footprint" "Package_SO:TSSOP-14_4.4x5mm_P0.65mm"
 			(at 90.17 43.18 0)
 			(effects
@@
 			)
 		)
-		(property "Footprint" "PCM_4ms_Resistor:R_Axial_DIN0207_L6.3mm_D2.5mm_P7.62mm_Horizontal"
+		(property "Footprint" "Resistor_SMD:R_0603_1608Metric"
 			(at 41.402 184.15 90)
 			(effects
@@
 			)
 		)
-		(property "Footprint" "Package_TO_SOT_THT:TO-92"
+		(property "Footprint" "Package_TO_SOT_SMD:SOT-23_Handsoldering"
 			(at 123.825 130.81 0)
 			(effects
@@
 			)
 		)
-		(property "Footprint" "Package_DIP:DIP-14_W7.62mm_Socket"
+		(property "Footprint" "Package_SO:SSOP-14_5.3x6.2mm_P0.65mm"
 			(at 143.51 128.27 0)
 			(effects
@@
 			)
 		)
-		(property "Footprint" "PCM_4ms_Resistor:R_Axial_DIN0207_L6.3mm_D2.5mm_P7.62mm_Horizontal"
+		(property "Footprint" "Resistor_SMD:R_0603_1608Metric"
 			(at 113.03 189.738 90)
 			(effects
