File: kicad/ida-button-smt/power.kicad_sch (KiCad schematic)
At the start: 18 parts, among them J4 EURO_PWR_2x5, U1 TL074, U2 40106, U3 L78L05_TO92, U4 TL074

Commit message: stylophone rev1
Parts:
- C10, C11, C12, C13, C5, C6, C9: footprint PCM_4ms_Capacitor:C_Disc_P5.08mm -> Capacitor_SMD:C_0603_1608Metric
- C2, C3: footprint PCM_4ms_Capacitor:CP_Radial_P2.5mm -> Capacitor_SMD:C_0603_1608Metric
- D3, D4: footprint PCM_4ms_Diode:D_DO-41_P7.62mm_Horizontal -> Diode_SMD:D_0603_1608Metric
- R4, R6: footprint PCM_4ms_Resistor:R_Axial_DIN0207_L6.3mm_D2.5mm_P7.62mm_Horizontal -> Resistor_SMD:R_0603_1608Metric
- U1, U4: footprint Package_DIP:DIP-14_W7.62mm_Socket -> Package_SO:SSOP-14_5.3x6.2mm_P0.65mm
- U2: footprint Package_DIP:DIP-14_W7.62mm_Socket -> Package_SO:TSSOP-14_4.4x5mm_P0.65mm
- U3: footprint Package_TO_SOT_THT:TO-92_Inline -> Package_TO_SOT_SMD:SOT-89-3_Handsoldering
Changed lines of the file:
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@@
 			)
 		)
-		(property "Footprint" "PCM_4ms_Diode:D_DO-41_P7.62mm_Horizontal"
+		(property "Footprint" "Diode_SMD:D_0603_1608Metric"
 			(at 53.34 64.135 0)
 			(effects
@@
 			)
 		)
-		(property "Footprint" "PCM_4ms_Diode:D_DO-41_P7.62mm_Horizontal"
+		(property "Footprint" "Diode_SMD:D_0603_1608Metric"
 			(at 53.34 26.035 0)
 			(effects
@@
 			)
 		)
-		(property "Footprint" "PCM_4ms_Capacitor:C_Disc_P5.08mm"
+		(property "Footprint" "Capacitor_SMD:C_0603_1608Metric"
 			(at 128.27 53.6448 0)
 			(effects
@@
 			)
 		)
-		(property "Footprint" "Package_TO_SOT_THT:TO-92_Inline"
+		(property "Footprint" "Package_TO_SOT_SMD:SOT-89-3_Handsoldering"
 			(at 38.1 73.025 0)
 			(effects
@@
 			)
 		)
-		(property "Footprint" "PCM_4ms_Capacitor:CP_Radial_P2.5mm"
+		(property "Footprint" "Capacitor_SMD:C_0603_1608Metric"
 			(at 65.0748 59.69 0)
 			(effects
@@
 			)
 		)
-		(property "Footprint" "Package_DIP:DIP-14_W7.62mm_Socket"
+		(property "Footprint" "Package_SO:SSOP-14_5.3x6.2mm_P0.65mm"
 			(at 121.92 43.18 0)
 			(effects
@@
 			)
 		)
-		(property "Footprint" "PCM_4ms_Capacitor:C_Disc_P5.08mm"
+		(property "Footprint" "Capacitor_SMD:C_0603_1608Metric"
 			(at 46.6852 90.17 0)
 			(effects
@@
 			)
 		)
-		(property "Footprint" "PCM_4ms_Capacitor:C_Disc_P5.08mm"
+		(property "Footprint" "Capacitor_SMD:C_0603_1608Metric"
 			(at 153.67 35.8648 0)
 			(effects
@@
 			)
 		)
-		(property "Footprint" "PCM_4ms_Capacitor:C_Disc_P5.08mm"
+		(property "Footprint" "Capacitor_SMD:C_0603_1608Metric"
 			(at 128.27 35.8648 0)
 			(effects
@@
 			)
 		)
-		(property "Footprint" "PCM_4ms_Resistor:R_Axial_DIN0207_L6.3mm_D2.5mm_P7.62mm_Horizontal"
+		(property "Footprint" "Resistor_SMD:R_0603_1608Metric"
 			(at 33.02 114.808 90)
 			(effects
@@
 			)
 		)
-		(property "Footprint" "Package_DIP:DIP-14_W7.62mm_Socket"
+		(property "Footprint" "Package_SO:SSOP-14_5.3x6.2mm_P0.65mm"
 			(at 147.32 43.18 0)
 			(effects
@@
 			)
 		)
-		(property "Footprint" "Package_DIP:DIP-14_W7.62mm_Socket"
+		(property "Footprint" "Package_SO:TSSOP-14_4.4x5mm_P0.65mm"
 			(at 93.98 44.45 0)
 			(effects
@@
 			)
 		)
-		(property "Footprint" "PCM_4ms_Capacitor:C_Disc_P5.08mm"
+		(property "Footprint" "Capacitor_SMD:C_0603_1608Metric"
 			(at 101.6 29.5148 0)
 			(effects
@@
 			)
 		)
-		(property "Footprint" "PCM_4ms_Resistor:R_Axial_DIN0207_L6.3mm_D2.5mm_P7.62mm_Horizontal"
+		(property "Footprint" "Resistor_SMD:R_0603_1608Metric"
 			(at 23.622 119.38 90)
 			(effects
@@
 			)
 		)
-		(property "Footprint" "PCM_4ms_Capacitor:C_Disc_P5.08mm"
+		(property "Footprint" "Capacitor_SMD:C_0603_1608Metric"
 			(at 31.4452 90.17 0)
 			(effects
@@
 			)
 		)
-		(property "Footprint" "PCM_4ms_Capacitor:C_Disc_P5.08mm"
+		(property "Footprint" "Capacitor_SMD:C_0603_1608Metric"
 			(at 153.67 53.6448 0)
 			(effects
@@
 			)
 		)
-		(property "Footprint" "PCM_4ms_Capacitor:CP_Radial_P2.5mm"
+		(property "Footprint" "Capacitor_SMD:C_0603_1608Metric"
 			(at 67.0052 40.64 0)
 			(effects
