File: kicad/noise/noise.kicad_pcb (KiCad board)
At the start: 2 copper layers, 19.9 x 100 mm, 30 parts, among them J1 EURO_PWR_2x5, J2 PINK, J3 WHITE, Q1 BC548, U1 TL072

Commit message: stylophone rev1
Parts:
- R1, R10, R11, R12, R2, R3, R4, R5, R6: footprint PCM_4ms_Resistor:R_0603 -> Resistor_SMD:R_0603_1608Metric
Routing:
- net Net-(R10-Pad2): track 5.74 -> 10.3 mm
- net Net-(U1B-+): track 53.1 -> 54.8 mm
- net Net-(U1B--): track 13.2 -> 12.1 mm
- net Net-(U1A--): track 11.2 -> 10.4 mm
