File: kicad/mixer/controls.kicad_sch (KiCad schematic)
At the start: 74 parts, among them J1 RETURN_L, J10 CH4_IN, J11 CH5_IN, J2 RETURN_R, J3 SEND_L, J4 SEND_R, J5 MIX_L, J6 MIX_R, J7 CH1_IN, J8 CH2_IN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

Commit message: been a minute huh
Parts:
- removed J1: RETURN_L, Connector_Audio:Jack_3.5mm_QingPu_WQP-PJ398SM_Vertical_CircularHoles, symbol Connector_Audio:AudioJack2_SwitchT
- removed J10: CH4_IN, Connector_Audio:Jack_3.5mm_QingPu_WQP-PJ398SM_Vertical_CircularHoles, symbol Connector_Audio:AudioJack2_SwitchT
- removed J11: CH5_IN, Connector_Audio:Jack_3.5mm_QingPu_WQP-PJ398SM_Vertical_CircularHoles, symbol Connector_Audio:AudioJack2_SwitchT
- removed J2: RETURN_R, Connector_Audio:Jack_3.5mm_QingPu_WQP-PJ398SM_Vertical_CircularHoles, symbol Connector_Audio:AudioJack2_SwitchT
- removed J4: SEND_R, Connector_Audio:Jack_3.5mm_QingPu_WQP-PJ398SM_Vertical_CircularHoles, symbol Connector_Audio:AudioJack2_SwitchT
- removed J7: CH1_IN, Connector_Audio:Jack_3.5mm_QingPu_WQP-PJ398SM_Vertical_CircularHoles, symbol Connector_Audio:AudioJack2_SwitchT
- removed J8: CH2_IN, Connector_Audio:Jack_3.5mm_QingPu_WQP-PJ398SM_Vertical_CircularHoles, symbol Connector_Audio:AudioJack2_SwitchT
- removed J9: CH3_IN, Connector_Audio:Jack_3.5mm_QingPu_WQP-PJ398SM_Vertical_CircularHoles, symbol Connector_Audio:AudioJack2_SwitchT
- removed R10, R11, R17, R18, R22, R26, R31, R32, R38, R42: 10k, Resistor_SMD:R_0603_1608Metric_Pad0.98x0.95mm_HandSolder, symbol Device:R
- removed R12, R13, R14, R15, R16, R19, R20, R21, R25, R29, R30, R33, R34, R35, R36, R37, R40, R41, R5, R6, R7, R8, R9: 100k, Resistor_SMD:R_0603_1608Metric_Pad0.98x0.95mm_HandSolder, symbol Device:R
- removed R44: 4k7, Resistor_SMD:R_0603_1608Metric_Pad0.98x0.95mm_HandSolder, symbol Device:R
- removed RV1, RV11, RV15, RV4, RV8: A10k, Potentiometer_THT:Potentiometer_Alpha_RD901F-40-00D_Single_Vertical, symbol Device:R_Potentiometer
- removed RV10, RV13, RV14, RV17, RV3, RV6: A10k, Potentiometer_THT:Potentiometer_Alpha_RD902F-40-00D_Dual_Vertical, symbol Device:R_Potentiometer_Dual_Separate
- removed RV12, RV16, RV2, RV5, RV9: B10k, Potentiometer_THT:Potentiometer_Alpha_RD901F-40-00D_Single_Vertical, symbol Device:R_Potentiometer
- removed U2: TL074, Package_SO:SSOP-14_5.3x6.2mm_P0.65mm, symbol KitsBlips:TL074
- added U2: TL072, Package_SO:SOIC-8_3.9x4.9mm_P1.27mm, symbol KitsBlips:TL072
- J3: value SEND_L -> SEND_OUT; footprint Connector_Audio:Jack_3.5mm_QingPu_WQP-PJ398SM_Vertical_CircularHoles -> KitsBlips:Jack_3.5mm_QingPu_WQP-PJ398SM_Vertical_CircularHoles
- J5, J6: footprint Connector_Audio:Jack_3.5mm_QingPu_WQP-PJ398SM_Vertical_CircularHoles -> KitsBlips:Jack_3.5mm_QingPu_WQP-PJ398SM_Vertical_CircularHoles
- R23, R28: value 4k7 -> 2k4
- R3: value 1k -> 10k
- R39: value 4k7 -> 3k3
- RV7: footprint Potentiometer_THT:Potentiometer_Alpha_RD902F-40-00D_Dual_Vertical -> KitsBlips:Potentiometer_Alpha_RD902F-40-00D_Dual_Vertical
- U1: footprint Package_SO:SSOP-14_5.3x6.2mm_P0.65mm -> Package_SO:SOIC-14_3.9x8.7mm_P1.27mm
Connections:
- net GND2: now also U2.3 (+), U2.5 (+)
- net at R39.1: now also R3.2, U2.6 (-)
- net at R4.2: now also R3.1, U2.7
- net at R39.2, R43.1: now also U2.1
- net SEND_L renamed SEND
- net SEND: now also U2.2 (-)
- no-connect marks 4 -> 2
Other:
- added sheet mono_channel (mono_channel.kicad_sch)
- added sheet mono_channel1 (mono_channel.kicad_sch)
- added sheet mono_channel2 (mono_channel.kicad_sch)
- added sheet mono_channel3 (mono_channel.kicad_sch)
- added sheet mono_channel4 (mono_channel.kicad_sch)
- note added: "All Mix/Send inputs expected to have effective resistance of 100k-130k"

Commit message: tweaks for embedding on blog
Other:
- note added: "All Mix/Send inputs expected to have 100k resistance"
- note removed: "All Mix/Send inputs expected to have effective resistance of 100k-130k"
Changed lines of the file:
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@@
+	)
+	(junction
+		(at 199.39 109.22)
+		(diameter 0)
+		(color 0 0 0 0)
 	)
 	(junction
@@
 		)
 	)
-	(text "All Mix/Send inputs expected to have effective resistance of 100k-130k"
+	(text "All Mix/Send inputs expected to have 100k resistance"
 		(exclude_from_sim no)
-		(at 226.568 22.098 0)
+		(at 153.67 24.892 0)
 		(effects
 			(font
