File: kicad/mixer/mixer.kicad_sch (KiCad schematic)
At the start: 0 parts

Commit message: tweaks for embedding on blog
Parts:
- added J1: MIX_L, KitsBlips:Jack_3.5mm_QingPu_WQP-PJ398SM_Vertical_CircularHoles, symbol Connector_Audio:AudioJack2_SwitchT
- added J2: MIX_R, KitsBlips:Jack_3.5mm_QingPu_WQP-PJ398SM_Vertical_CircularHoles, symbol Connector_Audio:AudioJack2_SwitchT
- added J3: SEND_OUT, KitsBlips:Jack_3.5mm_QingPu_WQP-PJ398SM_Vertical_CircularHoles, symbol Connector_Audio:AudioJack2_SwitchT
- added R1, R2, R3: 100k, Resistor_SMD:R_0603_1608Metric_Pad0.98x0.95mm_HandSolder, symbol Device:R
- added R10, R8, R9: 1k, Resistor_SMD:R_0603_1608Metric_Pad0.98x0.95mm_HandSolder, symbol Device:R
- added R4, R5: 2k4, Resistor_SMD:R_0603_1608Metric_Pad0.98x0.95mm_HandSolder, symbol Device:R
- added R6: 3k3, Resistor_SMD:R_0603_1608Metric_Pad0.98x0.95mm_HandSolder, symbol Device:R
- added R7: 10k, Resistor_SMD:R_0603_1608Metric_Pad0.98x0.95mm_HandSolder, symbol Device:R
- added RV1: A10k, KitsBlips:Potentiometer_Alpha_RD902F-40-00D_Dual_Vertical, symbol Device:R_Potentiometer_Dual_Separate
- added U1: TL074, Package_SO:SOIC-14_3.9x8.7mm_P1.27mm, symbol KitsBlips:TL074
- added U2: TL072, Package_SO:SOIC-8_3.9x4.9mm_P1.27mm, symbol KitsBlips:TL072
Connections:
- new net: R5.1, RV1.4, U1.13 (-)
- new net: R2.1, R5.2, U1.8
- new net: R1.1, R4.2, U1.1
- new net: J2.T, R9.1
- new net: R9.2, RV1.5, U1.14
- new net: R4.1, RV1.1, U1.6 (-)
- new net: R8.2, RV1.2, U1.7
- new net: J3.T, R10.1
- new net: R10.2, R7.1, U2.7
- new net: R6.1, R7.2, U2.6 (-)
- new net: R3.1, R6.2, U2.1
- new net: J1.T, R8.1
- new net GND2: J1.S, J2.S, J3.S, U1.10 (+), U1.12 (+), U1.3 (+), U1.5 (+), U2.3 (+), U2.5 (+)
- new net MIX_L: R1.2, U1.2 (-)
- new net MIX_R: R2.2, U1.9 (-)
- new net SEND: R3.2, U2.2 (-)
- no-connect marks 0 -> 5
Other:
- removed sheet controls
- added sheet mono_channel (mono_channel.kicad_sch)
- added sheet mono_channel1 (mono_channel.kicad_sch)
- added sheet mono_channel2 (mono_channel.kicad_sch)
- added sheet mono_channel3 (mono_channel.kicad_sch)
- added sheet mono_channel4 (mono_channel.kicad_sch)
- note added: "All Mix/Send inputs expected to have 100k resistance"
- note added: "Gain: x0 - x4.1"
- note added: "Gain: x3.0"
- title: (none) -> KB01 - KitsMix
