File: kicad/mixer/mono_channel.kicad_sch (KiCad schematic)
At the start: 10 parts, among them J2 MONO_IN

Commit message: tweaks for embedding on blog
Parts:
- renumbered J2 to J4, R17 to R11, R18 to R12, R19 to R13, R20 to R14, R21 to R15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
Connections:
- no-connect marks 0 -> 1
Other:
- title: (none) -> Mono input channel
- moved on the sheet: J4, R11, R12, R13, R14, R15, R16, RV2, RV3, RV4
